File: USB-Voltage-Probe-No-Slot/USB-Voltage-Probe.sch (KiCad schematic (older format))
At the start: 4 parts, among them J1 USB3_A, J2 USB3_A, J3 GND, J4 VBUS

Commit message: Created USB Power Cleaner that filters out switching noize
Parts:
- J1, J2: symbol Connector_Specialized:USB3_A -> Connector:USB3_A
Changed lines of the file:
@@
 $EndDescr
 $Comp
-L Connector_Specialized:USB3_A J1
+L Connector:USB3_A J1
 U 1 1 5B1E0CAE
 P 4200 2900
@@
 $EndComp
 $Comp
-L Connector_Specialized:USB3_A J2
+L Connector:USB3_A J2
 U 1 1 5B1E0DCF
 P 7200 2900
